Commit message: chang our base_scan position

File: omo_r1_description/urdf/omo_r1.urdf.xacro (robot description, xacro)
@@ -135,5 +135,5 @@
     <parent link="base_link"/>
     <child link="base_scan"/>
-    <origin xyz="0.06 0 0.230" rpy="0.0 0 3.14159"/>
+    <origin xyz="-0.15 0 1.2" rpy="0.0 0 3.14159"/>
   </joint>
   <link name="base_scan">
